File: eagle/midi_to_cv.brd (EAGLE design)
At the start: 100 x 80 mm, 57 parts, among them IC1 TL084P, IC2 TL084P, U1 ATMEGA328P_PDIP

Commit message: will add iscp header
Parts:
- added JP1: (no value), pinhead:2X03
Changed lines of the file:
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@@
 <element name="PAD21" library="wirepad" package="2,54/0,9" value="gate" x="27.94" y="38.1"/>
 <element name="PAD22" library="wirepad" package="2,54/0,9" value="gate" x="31.75" y="38.1"/>
+<element name="JP1" library="pinhead" package="2X03" value="" x="-5.08" y="5.08"/>
 </elements>
 <signals>
