File: eagle/midi_to_cv.brd (EAGLE design)
At the start: 100 x 80 mm, 49 parts, among them IC1 TL084P, IC2 TL084P, U1 ATMEGA328P_PDIP

Commit message: this interface is getting sirius
Parts:
- removed PAD10, PAD7, PAD8, PAD9: gate output, wirepad:2,54/0,9
- removed PAD11, PAD14: gate LED, wirepad:2,54/0,9
- removed PAD12: reset, wirepad:2,54/0,9
- added AUTOTUNE, DEL_TRIG, MOUT_P2, MOUT_P4, MOUT_P5, MTHRU_P2, MTHRU_P4, MTHRU_P5: pad, wirepad:2,54/0,9
- added C4: .01u, rcl:C050-024X044
- added C5, C6: .1uF, rcl:C025-040X050
- added D3: 1N4148DO35-10, diode:DO35-10
- added DELAY, DELAY1: (no value), pot:3RP/1610N
- added DELGATELED1, DELGATELED2, GATELED1, GATELED2, PIN13LED1, PIN13LED2: gate LED, wirepad:2,54/0,9
- added DEL_GATE, GATE: gate output, wirepad:2,54/0,9
- added IC3: 4067N, 40xx:DIL24-6
- added JP1: (no value), SparkFun-Connectors:2X3-NS
- added R24: 1M, rcl:0207/10
- added R25, R27: 1k, rcl:0207/10
- added R28: 10k, rcl:0207/10
- added RST1: reset, wirepad:2,54/0,9
- added T1, T2: 2N3904, transistor:TO92
- added U4: 4584N, TR808clone:DIL14
- BEND: value bend output -> pad
- IC2: value TL084P -> 4067N; device linear:DIL14 -> 40xx:DIL24-6
- MOD: value mod output -> pad
- PITCH: value pitch output -> pad
- R18: value 1k -> 10k
- R19, R21, R22, R23: value 1k -> 220
- R20: value 1k -> 100k
- VELOC: value velocity out -> pad
- moved R19 188.8 mm to (-1.27, -154.9), turned to 0 degrees
- moved R23 186.3 mm to (-11.4, -160.0), turned to 0 degrees
- moved R21 149.5 mm to (-1.27, -116.8)
- moved R22 148.3 mm to (-11.4, -121.9), turned to 0 degrees
- moved IC2 123.7 mm to (1.27, -95.2), turned to 0 degrees
- moved R20 105.1 mm to (6.35, -83.8), turned to 0 degrees
- moved R17 30.9 mm to (59.7, 17.8), turned to 0 degrees
- moved R4 28.0 mm to (66.0, 58.4)
- moved R16 19.1 mm to (44.5, 17.8), turned to 0 degrees
- moved R18 11.4 mm to (38.1, 22.9), turned to 90 degrees
- moved R10 9.67 mm to (54.6, 59.7)
- moved R5 8.98 mm to (43.2, 68.6)
- moved U$4 7.73 mm to (49.5, 63.5)
- renumbered PAD1 to MIDI_IN_4, PAD13 to RST2, PAD2 to MIDI_IN_5, PAD3 to PITCH, PAD4 to BEND, PAD5 to VELOC, PAD6 to MOD
Connections:
- removed net N$42: IC2.6, R17.1, R21.2
- new net N$43: JP1.5, R1.2, RST1.1, U1.1
- new net N$44: GATE.1, R27.2
- new net N$45: JP1.1, U$4.2, U1.18
- new net N$46: MOUT_P5.1, R19.2
- new net N$47: GATELED2.1, R25.2, R27.1
- new net N$48: C4.2, D3.C
- new net N$49: DEL_TRIG.1, U4.6
- new net N$50: R21.1, U4.2
- new net N$51: DELAY1.2, VELOC.1
- new net N$52: MTHRU_P5.1, R21.2
- new net N$54: MTHRU_P4.1, R22.2
- new net N$55: MOUT_P4.1, R23.2
- new net N$57: R19.1, U1.3
- net +12V: now also T1.1, T2.1; no longer IC2.4
- net +5V: now also C5.1, C6.1, DELAY.3, IC2.24, IC3.24, JP1.2, R22.1, R23.1, U4.14
- net -12V: no longer IC2.11
- net GND: now also C5.2, C6.2, DELAY.1, DELAY1.1, IC2.12, IC3.12, JP1.6, MOUT_P2.1, MTHRU_P2.1, PIN13LED1.1, R16.1, R18.1, R25.1, R28.1, U4.7; no longer PAD14.1, R21.1, R22.1, R23.1
- net N$1: now also GATELED1.1, T1.3; no longer PAD12.1, R1.2, U1.1
- net N$10: now also JP1.3
- net N$11: now also PIN13LED2.1; no longer PAD11.1
- net N$19: now also DELAY1.3; no longer VELOC.1
- net N$26: now also JP1.4
- net N$27: now also DELAY.2, U1.23; no longer U$4.2, U1.18
- net N$30: now also U4.9
- net N$31: now also DELGATELED1.1, T2.3; no longer IC2.3, U1.3
- net N$32: now also R18.2, T2.2; no longer IC2.5
- net N$33: now also R28.2, T1.2; no longer IC2.10
- net N$34: now also AUTOTUNE.1, U4.13; no longer IC2.12, U1.6
- net N$35: now also D3.A, DEL_GATE.1, R17.2; no longer IC2.1, PAD7.1, R16.2
- net N$36: now also DELGATELED2.1, R16.2, R17.1; no longer IC2.7, PAD8.1, R17.2
- net N$37: now also U4.11, U4.12; no longer IC2.8, PAD9.1, R18.2
- net N$38: now also U1.11, U4.10; no longer IC2.14, PAD10.1, R19.2
- net N$39: now also U4.1, U4.8; no longer IC2.2, R16.1, R20.2
- net N$4: now also R24.2
- net N$40: now also U4.4, U4.5; no longer IC2.13, R19.1, R23.2
- net N$41: now also C4.1, R20.2, U4.3; no longer IC2.9, R18.1, R22.2
- net N$5: now also R24.1

Commit message: updated gate circuits and normalled gate and cv to power connector and swapped vel and mod outputs
Parts:
- removed BEND: pad, wirepad:2,54/0,9
- removed DELGATELED1, DELGATELED2, GATELED1, GATELED2: gate LED, wirepad:2,54/0,9
- removed T1, T2: 2N3904, transistor:TO92
- added IC4: TL072P, linear:DIL08
- added LED1, LED2: (no value), SparkFun-LED:LED3MM
- added PRESSURE: pad, wirepad:2,54/0,9
- added R26, R29: 1k, rcl:0207/10
- AMT: value (none) -> 100k
- PIN13LED1, PIN13LED2: value gate LED -> activity LED
- R11: value 5k -> 1k
- R16, R25: value 1k -> 4.7k
- R17: value 1k -> 10k
- R18: value 10k -> 20k
- R27: value 1k -> 20k
- R4: value 10k -> 2k
- R8: value 3.3k -> 1k
- R9: value 10k -> 1k; device pot:B64W -> rcl:0207/10
- moved R9 263.6 mm to (-11.4, -185.4), turned to 0 degrees
- moved R10 258.8 mm to (-11.4, -190.5), turned to 0 degrees
- moved R28 247.9 mm to (-11.4, -215.9), turned to 0 degrees
- moved R27 237.2 mm to (-11.4, -210.8), turned to 0 degrees
- moved R18 228.9 mm to (-11.4, -200.7), turned to 0 degrees
- moved R17 224.9 mm to (-11.4, -195.6)
- moved VELOC 5.08 mm to (69.8, 54.6)
- renumbered DELAY1 to AMT
Connections:
- new net N$42: IC4.5, R10.1
- new net N$53: IC4.7, LED2.A, R29.2
- new net V+: IC4.8
- new net V-: IC4.4
- net +12V: now also R18.2, R27.2; no longer T1.1, T2.1
- net +5V: no longer R9.E
- net GND: now also R17.1, R8.1; no longer R18.1, R9.A
- net N$1: now also IC4.3, R9.1; no longer GATELED1.1, T1.3
- net N$14: now also IC1.5; no longer R10.1
- net N$15: now also IC4.2, R17.2, R18.1; no longer IC1.5, R10.2
- net N$16: now also IC4.1, LED1.A, R26.2; no longer R8.1, R9.S
- net N$17: now also AMT.3; no longer BEND.1
- net N$19: now also PRESSURE.1; no longer AMT.3
- net N$31: now also GATE.1, R26.1, U$1.15, U$1.16; no longer DELGATELED1.1, T2.3
- net N$32: now also R10.2; no longer R18.2, T2.2
- net N$33: now also R9.2; no longer R28.2, T1.2
- net N$35: now also R29.1; no longer R17.2
- net N$36: now also LED2.K; no longer DELGATELED2.1, R17.1
- net N$44: now also IC4.6, R27.1, R28.2; no longer GATE.1, R27.2
- net N$47: now also LED1.K; no longer GATELED2.1, R27.1
- net N$9: now also U$1.13, U$1.14
